File: pcb5.kicad_pcb (KiCad board)
At the start: 2 copper layers, 68.5 x 53 mm, 66 parts, among them J1 Conn_01x03_Male, J2 Conn_01x03_Male, J3 Conn_01x10_Male, J4 Conn_01x03_Male, J5 Conn_01x02_Male, J6 Conn_01x10_Male, J7 Conn_01x01_Male, P1 AD8402ARUZ1, SW1 SW_Push, U1 LD1117V33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

Commit message: Changed design rule to make DRC not whine about diode
Other:
- net class Default: clearance 0.1 -> 0.05
- rule trace_clearance: 0.1 -> 0.05
Changed lines of the file:
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@@
   (setup
     (last_trace_width 0.25)
-    (trace_clearance 0.1)
+    (trace_clearance 0.05)
     (zone_clearance 0.508)
     (zone_45_only no)
@@
   (net 48 "Net-(R25-Pad1)")
   (net_class Default "This is the default net class."
-    (clearance 0.1)
+    (clearance 0.05)
     (trace_width 0.25)
     (via_dia 0.6)
@@
   (segment (start 137.0294 125.1891) (end 127.96 125.1891) (width 0.25) (layer F.Cu) (net 36))
   (segment (start 127.96 125.1891) (end 127.8382 125.3109) (width 0.25) (layer F.Cu) (net 36))
-  (segment (start 137.0294 124.5391) (end 137.9064 124.5391) (width 0.25) (layer F.Cu) (net 37) (status 400000))
+  (segment (start 137.0294 124.5391) (end 137.9064 124.5391) (width 0.25) (layer F.Cu) (net 37))
   (segment (start 145.669 113.03) (end 138.176 120.523) (width 0.25) (layer F.Cu) (net 37) (status 80000))
   (segment (start 145.669 112.522) (end 145.669 113.03) (width 0.25) (layer F.Cu) (net 37) (status 80000))

Commit message: New gerbers
Other:
- board text added: "Circuit Design by Lonnie Souder II Layout by Chris Dietsch"
Changed lines of the file:
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@@
-(kicad_pcb (version 4) (host pcbnew 4.0.7)
+(kicad_pcb (version 4) (host pcbnew 4.0.4-stable)
   (general
     (links 151)
     (no_connects 2)
-    (area 109.093 90.043 177.8 144.653)
+    (area 109.144999 90.213 177.748001 144.664501)
     (thickness 1.6)
-    (drawings 5)
+    (drawings 6)
     (tracks 1244)
     (zones 0)
@@
     (visible_elements 7FFFFF9F)
     (pcbplotparams
-      (layerselection 0x00030_80000001)
-      (usegerberextensions false)
+      (layerselection 0x010f0_80000001)
+      (usegerberextensions true)
       (excludeedgelayer true)
       (linewidth 0.100000)
@@
       (psa4output false)
       (plotreference true)
-      (plotvalue true)
+      (plotvalue false)
       (plotinvisibletext false)
       (padsonsilk false)
@@
       (outputformat 1)
       (mirror false)
-      (drillshape 1)
+      (drillshape 0)
       (scaleselection 1)
-      (outputdirectory ""))
+      (outputdirectory Gerbers2))
   )
   (net 0 "")
@@
     )
   )
+  (gr_text "Circuit Design by Lonnie Souder II\nLayout by Chris Dietsch" (at 110.303 142.0215) (layer F.SilkS)
+    (effects (font (size 1 1) (thickness 0.2)) (justify left))
+  )
   (gr_line (start 109.22 91.6305) (end 177.673 91.6305) (angle 90) (layer Edge.Cuts) (width 0.15))
   (gr_line (start 109.22 144.5895) (end 109.22 91.6305) (angle 90) (layer Edge.Cuts) (width 0.15))
@@
   (segment (start 132.7404 122.7709) (end 127.8382 122.7709) (width 0.25) (layer F.Cu) (net 37))
   (segment (start 134.5086 124.5391) (end 132.7404 122.7709) (width 0.25) (layer F.Cu) (net 37))
+  (segment (start 130.3274 140.2715) (end 130.4036 140.1953) (width 0.25) (layer F.Cu) (net 38))
+  (segment (start 125.984 140.2715) (end 130.3274 140.2715) (width 0.25) (layer F.Cu) (net 38))
+  (segment (start 125.1712 139.4587) (end 125.984 140.2715) (width 0.25) (layer F.Cu) (net 38))
   (segment (start 127.8382 120.2309) (end 126.8984 120.2309) (width 0.25) (layer F.Cu) (net 38))
   (segment (start 155.418 117.5431) (end 155.418 115.9347) (width 0.25) (layer F.Cu) (net 38))
@@
   (segment (start 130.4036 136.8933) (end 137.5156 129.7813) (width 0.25) (layer F.Cu) (net 38))
   (segment (start 130.4036 140.1953) (end 130.4036 136.8933) (width 0.25) (layer F.Cu) (net 38))
-  (segment (start 130.3274 140.2715) (end 130.4036 140.1953) (width 0.25) (layer F.Cu) (net 38))
-  (segment (start 125.984 140.2715) (end 130.3274 140.2715) (width 0.25) (layer F.Cu) (net 38))
-  (segment (start 125.1712 139.4587) (end 125.984 140.2715) (width 0.25) (layer F.Cu) (net 38))
   (segment (start 125.1712 121.9581) (end 125.1712 139.4587) (width 0.25) (layer F.Cu) (net 38))
   (segment (start 126.8984 120.2309) (end 125.1712 121.9581) (width 0.25) (layer F.Cu) (net 38))
